File: Weight-O-Matic_HW/Weight-O-Matic_HW.kicad_sch (KiCad schematic)
At the start: 14 parts, among them J1 XT30_Plug, J2 BJ_2.1x5.5mm, J5 USB_B_Mini_Receptacle, J6 4P4C_Receptacle, SW2 SW_SPST, SW3 SW_SP3T

Commit message: small adjustments
Parts:
- added C1: 10uF, symbol Device:C_Polarized
- added D1: ~, symbol Device:D
- A1: value Arduino_Nano_Every -> Arduino_Nano (AtMega 328P)
Connections:
- net +24V: now also C1.1
- net GND: now also C1.2
- net at J1. (-), M4. (NO): now also D1.2 (A)
- new net: D1.1 (K), J1. (-), M4. (NO)
